Commit message: start adding legs

File: bd1_description/urdf/bd1.xacro (robot description, xacro)
@@ -1,29 +1,51 @@
 <?xml version="1.0"?>
 <robot xmlns:xacro="http://www.ros.org/wiki/xacro" name="BD1" >
-    <xacro:property name="head_x" value="-0.05"/>
-    <xacro:property name="head_z" value="0.05"/>
+    <xacro:include filename="$(find bd1_description)/urdf/bd1_leg.xacro"/>
+    <xacro:property name="body_aprox_x" value="0.18"/>
+    <xacro:property name="body_aprox_y" value="0.12"/>
+    <xacro:property name="body_aprox_z" value="0.13"/>
+    <xacro:property name="body_mass" value="0.5"/>
+    <xacro:property name="head_aprox_x" value="0.29"/>
+    <xacro:property name="head_aprox_y" value="0.24"/>
+    <xacro:property name="head_aprox_z" value="0.1"/>
+    <xacro:property name="head_mass" value="0.5"/>
+    <xacro:property name="head_x_offset" value="-0.05"/>
+    <xacro:property name="head_z_offset" value="0.1"/>
     <xacro:property name="legs_baseline" value="0.2"/>
+    <link name="base_link">
+    </link>
+    <!--
+        BODY
+    -->
     <link name="body_link">
         <visual>
             <geometry>
                 <mesh filename="file://$(find bd1_description)/mesh/body_m.dae"/>
-                <!--<cylinder length="0.6" radius="0.2"/>-->
             </geometry>
         </visual>
         <collision>
+            <origin xyz="-0.02 0 0.005" rpy=" 0 0 0"/>
             <geometry>
-                <box size="0.1 0.1 0.1"/>
+                <box size="${body_aprox_x} ${body_aprox_y} ${body_aprox_z}"/>
             </geometry>
         </collision>
         <inertial>
-            <mass value="10.0"/>
-            <origin xyz="0.0 0 0.1" rpy=" 0 0 0"/>
+            <mass value="${body_mass}"/>
+            <!--<origin xyz="0.0 0 0.1" rpy=" 0 0 0"/>-->
             <inertia
-                ixx="0.5" ixy="0" ixz="0"
-                iyy="1.0" iyz="0"
-                izz="0.1"
+                ixx="${0.08*body_mass*(body_aprox_y*body_aprox_y+body_aprox_z*body_aprox_z)}" ixy="0" ixz="0"
+                iyy="${0.08*body_mass*(body_aprox_x*body_aprox_x+body_aprox_z*body_aprox_z)}" iyz="0"
+                izz="${0.08*body_mass*(body_aprox_x*body_aprox_x+body_aprox_y*body_aprox_y)}"
             />
         </inertial>
     </link>
+    <joint name="body_j" type="fixed">
+        <parent link="base_link"/>
+        <child link="body_link"/>
+        <origin xyz="0 0 0" rpy="0 0 0"/>
+    </joint>
+    <!--
+        HEAD
+    -->
     <link name="head_link">
         <visual>
@@ -33,15 +55,16 @@
         </visual>
         <collision>
+            <origin xyz="0.04 0 0.07" rpy=" 0 0 0"/>
             <geometry>
-                <box size="0.1 0.1 0.1"/>
+                <box size="${head_aprox_x} ${head_aprox_y} ${head_aprox_z}"/>
             </geometry>
         </collision>
         <inertial>
-            <mass value="10.0"/>
-            <origin xyz="0.0 0 0.1" rpy=" 0 0 0"/>
+            <mass value="${head_mass}"/>
+            <!--<origin xyz="0.0 0 0.1" rpy=" 0 0 0"/>-->
             <inertia
-                ixx="0.5" ixy="0" ixz="0"
-                iyy="1.0" iyz="0"
-                izz="0.1"
+                ixx="${0.08*head_mass*(head_aprox_y*head_aprox_y+head_aprox_z*head_aprox_z)}" ixy="0" ixz="0"
+                iyy="${0.08*head_mass*(head_aprox_x*head_aprox_x+head_aprox_z*head_aprox_z)}" iyz="0"
+                izz="${0.08*head_mass*(head_aprox_x*head_aprox_x+head_aprox_y*head_aprox_y)}"
             />
         </inertial>
@@ -50,5 +73,10 @@
         <parent link="body_link"/>
         <child link="head_link"/>
-        <origin xyz="${head_x} 0 ${head_z}" rpy="0 0 0"/>
+        <origin xyz="${head_x_offset} 0 ${head_z_offset}" rpy="0 0 0"/>
     </joint>
+    <!--
+        LEGS
+    -->
+    <xacro:bd1_leg side="r" y_offset="${-legs_baseline/2}"/>
+    <xacro:bd1_leg side="l" y_offset="${legs_baseline/2}"/>
 </robot>

Commit message: legs expanded

File: bd1_description/urdf/bd1.xacro (robot description, xacro)
@@ -12,5 +12,4 @@
     <xacro:property name="head_x_offset" value="-0.05"/>
     <xacro:property name="head_z_offset" value="0.1"/>
-    <xacro:property name="legs_baseline" value="0.2"/>
     <link name="base_link">
     </link>
@@ -78,5 +77,5 @@
         LEGS
     -->
-    <xacro:bd1_leg side="r" y_offset="${-legs_baseline/2}"/>
-    <xacro:bd1_leg side="l" y_offset="${legs_baseline/2}"/>
+    <xacro:bd1_leg side="r" y_mul="-1"/>
+    <xacro:bd1_leg side="l" y_mul="1"/>
 </robot>

File: bd1_description/urdf/bd1_leg.xacro (robot description, xacro)
@@ -1,9 +1,17 @@
 <?xml version="1.0"?>
 <robot xmlns:xacro="http://ros.org/wiki/xacro">
+    <xacro:property name="legs_baseline" value="0.2"/>
     <xacro:property name="up_leg_aprox_x" value="0.24"/>
     <xacro:property name="up_leg_aprox_y" value="0.05"/>
     <xacro:property name="up_leg_aprox_z" value="0.12"/>
     <xacro:property name="up_leg_mass" value="0.25"/>
-    <xacro:macro name="bd1_leg" params="side y_offset">
+    <xacro:property name="mid_leg_aprox_x" value="0.24"/>
+    <xacro:property name="mid_leg_aprox_y" value="0.05"/>
+    <xacro:property name="mid_leg_aprox_z" value="0.12"/>
+    <xacro:property name="mid_leg_mass" value="0.25"/>
+    <xacro:macro name="bd1_leg" params="side y_mul">
+        <!--
+        UP
+        -->
         <link name="up_leg_${side}_link">
             <visual>
@@ -13,5 +21,5 @@
             </visual>
             <collision>
-                <origin xyz="0.08 0.02 0.0" rpy=" 0 0 0"/>
+                <origin xyz="0.08 ${y_mul*0.02} 0.0" rpy=" 0 0 0"/>
                 <geometry>
                     <box size="${up_leg_aprox_x} ${up_leg_aprox_y} ${up_leg_aprox_z}"/>
@@ -31,5 +39,35 @@
             <parent link="body_link"/>
             <child link="up_leg_${side}_link"/>
-            <origin xyz="0 ${y_offset} 0" rpy="0 ${pi/2} 0"/>
+            <origin xyz="0 ${y_mul*legs_baseline/2} 0" rpy="0 ${pi/2} 0"/>
+        </joint>
+        <!--
+        MID
+        -->
+        <link name="mid_leg_${side}_link">
+            <visual>
+                <geometry>
+                    <mesh filename="file://$(find bd1_description)/mesh/mid_leg_${side}_m.dae"/>
+                </geometry>
+            </visual>
+            <collision>
+                <origin xyz="-0.08 ${y_mul*0.02} 0.0" rpy=" 0 0 0"/>
+                <geometry>
+                    <box size="${mid_leg_aprox_x} ${mid_leg_aprox_y} ${mid_leg_aprox_z}"/>
+                </geometry>
+            </collision>
+            <inertial>
+                <mass value="${mid_leg_mass}"/>
+                <!--<origin xyz="0.0 0 0.1" rpy=" 0 0 0"/>-->
+                <inertia
+                    ixx="${0.08*mid_leg_mass*(mid_leg_aprox_y*mid_leg_aprox_y+mid_leg_aprox_z*mid_leg_aprox_z)}" ixy="0" ixz="0"
+                    iyy="${0.08*mid_leg_mass*(mid_leg_aprox_x*mid_leg_aprox_x+mid_leg_aprox_z*mid_leg_aprox_z)}" iyz="0"
+                    izz="${0.08*mid_leg_mass*(mid_leg_aprox_y*mid_leg_aprox_y+mid_leg_aprox_x*mid_leg_aprox_x)}"
+                />
+            </inertial>
+        </link>
+        <joint name="mid_leg_${side}_j" type="fixed">
+            <parent link="up_leg_${side}_link"/>
+            <child link="mid_leg_${side}_link"/>
+            <origin xyz="0.15 ${-y_mul*0.05} 0" rpy="0 ${pi} 0"/>
         </joint>
     </xacro:macro>

Commit message: up leg parts looks ok

File: bd1_description/urdf/bd1.xacro (robot description, xacro)
@@ -24,5 +24,5 @@
         </visual>
         <collision>
-            <origin xyz="-0.02 0 0.005" rpy=" 0 0 0"/>
+            <origin xyz="-0.015 0 0.005" rpy=" 0 0 0"/>
             <geometry>
                 <box size="${body_aprox_x} ${body_aprox_y} ${body_aprox_z}"/>

File: bd1_description/urdf/bd1_leg.xacro (robot description, xacro)
@@ -1,5 +1,5 @@
 <?xml version="1.0"?>
 <robot xmlns:xacro="http://ros.org/wiki/xacro">
-    <xacro:property name="legs_baseline" value="0.2"/>
+    <xacro:property name="legs_baseline" value="0.12"/>
     <xacro:property name="up_leg_aprox_x" value="0.24"/>
     <xacro:property name="up_leg_aprox_y" value="0.05"/>
@@ -21,5 +21,5 @@
             </visual>
             <collision>
-                <origin xyz="0.08 ${y_mul*0.02} 0.0" rpy=" 0 0 0"/>
+                <origin xyz="0.065 ${y_mul*0.03} 0.0" rpy=" 0 0 0"/>
                 <geometry>
                     <box size="${up_leg_aprox_x} ${up_leg_aprox_y} ${up_leg_aprox_z}"/>

Commit message: mid leg is ok

File: bd1_description/urdf/bd1.xacro (robot description, xacro)
@@ -31,5 +31,4 @@
         <inertial>
             <mass value="${body_mass}"/>
-            <!--<origin xyz="0.0 0 0.1" rpy=" 0 0 0"/>-->
             <inertia
                 ixx="${0.08*body_mass*(body_aprox_y*body_aprox_y+body_aprox_z*body_aprox_z)}" ixy="0" ixz="0"
@@ -61,5 +60,4 @@
         <inertial>
             <mass value="${head_mass}"/>
-            <!--<origin xyz="0.0 0 0.1" rpy=" 0 0 0"/>-->
             <inertia
                 ixx="${0.08*head_mass*(head_aprox_y*head_aprox_y+head_aprox_z*head_aprox_z)}" ixy="0" ixz="0"

File: bd1_description/urdf/bd1_leg.xacro (robot description, xacro)
@@ -3,10 +3,10 @@
     <xacro:property name="legs_baseline" value="0.12"/>
     <xacro:property name="up_leg_aprox_x" value="0.24"/>
-    <xacro:property name="up_leg_aprox_y" value="0.05"/>
+    <xacro:property name="up_leg_aprox_y" value="0.04"/>
     <xacro:property name="up_leg_aprox_z" value="0.12"/>
     <xacro:property name="up_leg_mass" value="0.25"/>
-    <xacro:property name="mid_leg_aprox_x" value="0.24"/>
-    <xacro:property name="mid_leg_aprox_y" value="0.05"/>
-    <xacro:property name="mid_leg_aprox_z" value="0.12"/>
+    <xacro:property name="mid_leg_aprox_x" value="0.22"/>
+    <xacro:property name="mid_leg_aprox_y" value="0.02"/>
+    <xacro:property name="mid_leg_aprox_z" value="0.08"/>
     <xacro:property name="mid_leg_mass" value="0.25"/>
     <xacro:macro name="bd1_leg" params="side y_mul">
@@ -28,5 +28,4 @@
             <inertial>
                 <mass value="${up_leg_mass}"/>
-                <!--<origin xyz="0.0 0 0.1" rpy=" 0 0 0"/>-->
                 <inertia
                     ixx="${0.08*up_leg_mass*(up_leg_aprox_y*up_leg_aprox_y+up_leg_aprox_z*up_leg_aprox_z)}" ixy="0" ixz="0"
@@ -51,5 +50,5 @@
             </visual>
             <collision>
-                <origin xyz="-0.08 ${y_mul*0.02} 0.0" rpy=" 0 0 0"/>
+                <origin xyz="0.07 ${-y_mul*0.01} 0.0" rpy=" 0 0 0"/>
                 <geometry>
                     <box size="${mid_leg_aprox_x} ${mid_leg_aprox_y} ${mid_leg_aprox_z}"/>
@@ -58,5 +57,4 @@
             <inertial>
                 <mass value="${mid_leg_mass}"/>
-                <!--<origin xyz="0.0 0 0.1" rpy=" 0 0 0"/>-->
                 <inertia
                     ixx="${0.08*mid_leg_mass*(mid_leg_aprox_y*mid_leg_aprox_y+mid_leg_aprox_z*mid_leg_aprox_z)}" ixy="0" ixz="0"
@@ -69,5 +67,5 @@
             <parent link="up_leg_${side}_link"/>
             <child link="mid_leg_${side}_link"/>
-            <origin xyz="0.15 ${-y_mul*0.05} 0" rpy="0 ${pi} 0"/>
+            <origin xyz="0.15 ${y_mul*0.009} 0" rpy="0 0 0"/>
         </joint>
     </xacro:macro>

Commit message: visual and collisions done

File: bd1_description/urdf/bd1.xacro (robot description, xacro)
@@ -22,4 +22,7 @@
                 <mesh filename="file://$(find bd1_description)/mesh/body_m.dae"/>
             </geometry>
+            <material name="white">
+                <color rgba="1 1 1 1"/>
+            </material>
         </visual>
         <collision>
@@ -51,4 +54,7 @@
                 <mesh filename="file://$(find bd1_description)/mesh/head_m.dae"/>
             </geometry>
+            <material name="white">
+                <color rgba="1 1 1 1"/>
+            </material>
         </visual>
         <collision>

File: bd1_description/urdf/bd1_leg.xacro (robot description, xacro)
@@ -10,4 +10,8 @@
     <xacro:property name="mid_leg_aprox_z" value="0.08"/>
     <xacro:property name="mid_leg_mass" value="0.25"/>
+    <xacro:property name="feet_aprox_x" value="0.25"/>
+    <xacro:property name="feet_aprox_y" value="0.06"/>
+    <xacro:property name="feet_aprox_z" value="0.025"/>
+    <xacro:property name="feet_mass" value="0.25"/>
     <xacro:macro name="bd1_leg" params="side y_mul">
         <!--
@@ -19,4 +23,7 @@
                     <mesh filename="file://$(find bd1_description)/mesh/up_leg_${side}_m.dae"/>
                 </geometry>
+                <material name="white">
+                <color rgba="1 1 1 1"/>
+            </material>
             </visual>
             <collision>
@@ -48,4 +55,7 @@
                     <mesh filename="file://$(find bd1_description)/mesh/mid_leg_${side}_m.dae"/>
                 </geometry>
+                <material name="white">
+                    <color rgba="1 1 1 1"/>
+                </material>
             </visual>
             <collision>
@@ -69,4 +79,36 @@
             <origin xyz="0.15 ${y_mul*0.009} 0" rpy="0 0 0"/>
         </joint>
+        <!--
+        FEET
+        -->
+        <link name="feet_${side}_link">
+            <visual>
+                <geometry>
+                    <mesh filename="file://$(find bd1_description)/mesh/feet_m.dae"/>
+                </geometry>
+                <material name="white">
+                    <color rgba="1 1 1 1"/>
+                </material>
+            </visual>
+            <collision>
+                <origin xyz="0.02 ${-y_mul*0.0} -0.065" rpy=" 0 0 0"/>
+                <geometry>
+                    <box size="${feet_aprox_x} ${feet_aprox_y} ${feet_aprox_z}"/>
+                </geometry>
+            </collision>
+            <inertial>
+                <mass value="${feet_mass}"/>
+                <inertia
+                    ixx="${0.08*feet_mass*(feet_aprox_y*feet_aprox_y+feet_aprox_z*feet_aprox_z)}" ixy="0" ixz="0"
+                    iyy="${0.08*feet_mass*(feet_aprox_x*feet_aprox_x+feet_aprox_z*feet_aprox_z)}" iyz="0"
+                    izz="${0.08*feet_mass*(feet_aprox_y*feet_aprox_y+feet_aprox_x*feet_aprox_x)}"
+                />
+            </inertial>
+        </link>
+        <joint name="feet_${side}_j" type="fixed">
+            <parent link="mid_leg_${side}_link"/>
+            <child link="feet_${side}_link"/>
+            <origin xyz="0.15 ${-y_mul*0.0045} 0" rpy="0 ${-pi/2} 0"/>
+        </joint>
     </xacro:macro>
 </robot>

Commit message: neck servo doesnot work

File: bd1_description/urdf/bd1.xacro (robot description, xacro)
@@ -9,7 +9,21 @@
     <xacro:property name="head_aprox_y" value="0.24"/>
     <xacro:property name="head_aprox_z" value="0.1"/>
-    <xacro:property name="head_mass" value="0.5"/>
+    <xacro:property name="head_mass" value="0.01"/>
     <xacro:property name="head_x_offset" value="-0.05"/>
     <xacro:property name="head_z_offset" value="0.1"/>
+    <!--
+    COMMON
+    -->
+    <xacro:macro name="servtransmission" params="joint">
+        <transmission name="${joint}_transm">
+            <type>transmission_interface/SimpleTransmission</type>
+            <joint name="${joint}">
+                <hardwareInterface>hardware_interface/PositionJointInterface</hardwareInterface>
+            </joint>
+            <actuator name="${joint}_motor">
+                <hardwareInterface>hardware_interface/PositionActuatorInterface</hardwareInterface>
+            </actuator>
+        </transmission>
+    </xacro:macro>
     <link name="base_link">
     </link>
@@ -47,4 +61,17 @@
     </joint>
     <!--
+        NECK
+    -->
+    <link name="neck_link">
+    </link>
+    <joint name="neck_j" type="revolute">
+        <parent link="body_link"/>
+        <child link="neck_link"/>
+        <origin xyz="0.02 0 0.02" rpy="0 0 0"/>
+        <limit effort="300000" velocity="0.1" lower="${-pi/2}" upper="${pi/2}"/>
+        <axis xyz="0 1 0"/>
+    </joint>
+    <xacro:servtransmission joint="neck_j"/>
+    <!--
         HEAD
     -->
@@ -74,7 +101,7 @@
     </link>
     <joint name="head_j" type="fixed">
-        <parent link="body_link"/>
+        <parent link="neck_link"/>
         <child link="head_link"/>
-        <origin xyz="${head_x_offset} 0 ${head_z_offset}" rpy="0 0 0"/>
+        <origin xyz="0 0 ${head_z_offset}" rpy="0 0 0"/>
     </joint>
     <!--

Commit message: neck worked

File: bd1_description/urdf/bd1.xacro (robot description, xacro)
@@ -2,4 +2,5 @@
 <robot xmlns:xacro="http://www.ros.org/wiki/xacro" name="BD1" >
     <xacro:include filename="$(find bd1_description)/urdf/bd1_leg.xacro"/>
+    <xacro:include filename="$(find bd1_description)/urdf/bd1.gazebo"/>
     <xacro:property name="body_aprox_x" value="0.18"/>
     <xacro:property name="body_aprox_y" value="0.12"/>
@@ -35,4 +36,5 @@
             <geometry>
                 <mesh filename="file://$(find bd1_description)/mesh/body_m.dae"/>
+                <!--<box size="${body_aprox_x} ${body_aprox_y} ${body_aprox_z}"/>-->
             </geometry>
             <material name="white">
@@ -69,5 +71,5 @@
         <child link="neck_link"/>
         <origin xyz="0.02 0 0.02" rpy="0 0 0"/>
-        <limit effort="300000" velocity="0.1" lower="${-pi/2}" upper="${pi/2}"/>
+        <limit effort="3000" velocity="0.1" lower="${-pi/2}" upper="${pi/2}"/>
         <axis xyz="0 1 0"/>
     </joint>
@@ -80,4 +82,5 @@
             <geometry>
                 <mesh filename="file://$(find bd1_description)/mesh/head_m.dae"/>
+                <!--<box size="${head_aprox_x} ${head_aprox_y} ${head_aprox_z}"/>-->
             </geometry>
             <material name="white">

File: bd1_description/urdf/bd1_leg.xacro (robot description, xacro)
@@ -22,4 +22,5 @@
                 <geometry>
                     <mesh filename="file://$(find bd1_description)/mesh/up_leg_${side}_m.dae"/>
+                    <!--<box size="${up_leg_aprox_x} ${up_leg_aprox_y} ${up_leg_aprox_z}"/>-->
                 </geometry>
                 <material name="white">
@@ -54,4 +55,5 @@
                 <geometry>
                     <mesh filename="file://$(find bd1_description)/mesh/mid_leg_${side}_m.dae"/>
+                    <!--<box size="${mid_leg_aprox_x} ${mid_leg_aprox_y} ${mid_leg_aprox_z}"/>-->
                 </geometry>
                 <material name="white">
@@ -86,4 +88,5 @@
                 <geometry>
                     <mesh filename="file://$(find bd1_description)/mesh/feet_m.dae"/>
+                    <!--<box size="${feet_aprox_x} ${feet_aprox_y} ${feet_aprox_z}"/>-->
                 </geometry>
                 <material name="white">
