Commit message: up leg part with servo, but rides like skies

File: bd1_description/urdf/bd1.xacro (robot description, xacro)
@@ -7,24 +7,18 @@
     <xacro:property name="body_aprox_z" value="0.13"/>
     <xacro:property name="body_mass" value="0.5"/>
+    <xacro:property name="neck_aprox_x" value="0.1"/>
+    <xacro:property name="neck_aprox_y" value="0.1"/>
+    <xacro:property name="neck_aprox_z" value="0.1"/>
+    <xacro:property name="neck_mass" value="0.01"/>
     <xacro:property name="head_aprox_x" value="0.29"/>
     <xacro:property name="head_aprox_y" value="0.24"/>
     <xacro:property name="head_aprox_z" value="0.1"/>
-    <xacro:property name="head_mass" value="0.01"/>
+    <xacro:property name="head_mass" value="0.5"/>
     <xacro:property name="head_x_offset" value="-0.05"/>
     <xacro:property name="head_z_offset" value="0.1"/>
+    <xacro:property name="servo_velocity" value="0.5"/>
     <!--
-    COMMON
+        BASE
     -->
-    <xacro:macro name="servtransmission" params="joint">
-        <transmission name="${joint}_transm">
-            <type>transmission_interface/SimpleTransmission</type>
-            <joint name="${joint}">
-                <hardwareInterface>hardware_interface/PositionJointInterface</hardwareInterface>
-            </joint>
-            <actuator name="${joint}_motor">
-                <hardwareInterface>hardware_interface/PositionActuatorInterface</hardwareInterface>
-            </actuator>
-        </transmission>
-    </xacro:macro>
     <link name="base_link">
     </link>
@@ -66,4 +60,12 @@
     -->
     <link name="neck_link">
+        <inertial>
+            <mass value="${neck_mass}"/>
+            <inertia
+                ixx="${0.08*neck_mass*(neck_aprox_y*neck_aprox_y+neck_aprox_z*neck_aprox_z)}" ixy="0" ixz="0"
+                iyy="${0.08*neck_mass*(neck_aprox_x*neck_aprox_x+neck_aprox_z*neck_aprox_z)}" iyz="0"
+                izz="${0.08*neck_mass*(neck_aprox_x*neck_aprox_x+neck_aprox_y*neck_aprox_y)}"
+            />
+        </inertial>
     </link>
     <joint name="neck_j" type="revolute">
@@ -71,5 +73,5 @@
         <child link="neck_link"/>
         <origin xyz="0.02 0 0.02" rpy="0 0 0"/>
-        <limit effort="3000" velocity="0.1" lower="${-pi/2}" upper="${pi/2}"/>
+        <limit effort="30" velocity="${servo_velocity}" lower="${-pi/2}" upper="${pi/2}"/>
         <axis xyz="0 1 0"/>
     </joint>
@@ -103,13 +105,16 @@
         </inertial>
     </link>
-    <joint name="head_j" type="fixed">
+    <joint name="head_j" type="revolute">
         <parent link="neck_link"/>
         <child link="head_link"/>
         <origin xyz="0 0 ${head_z_offset}" rpy="0 0 0"/>
+        <limit effort="30" velocity="${servo_velocity}" lower="${-pi/2}" upper="${pi/2}"/>
+        <axis xyz="0 1 0"/>
     </joint>
+    <xacro:servtransmission joint="head_j"/>
     <!--
         LEGS
     -->
-    <xacro:bd1_leg side="r" y_mul="-1"/>
-    <xacro:bd1_leg side="l" y_mul="1"/>
+    <xacro:bd1_leg side="r" y_mul="-1" servo_velocity="${servo_velocity}"/>
+    <xacro:bd1_leg side="l" y_mul="1" servo_velocity="${servo_velocity}"/>
 </robot>

File: bd1_description/urdf/bd1_leg.xacro (robot description, xacro)
@@ -14,5 +14,22 @@
     <xacro:property name="feet_aprox_z" value="0.025"/>
     <xacro:property name="feet_mass" value="0.25"/>
-    <xacro:macro name="bd1_leg" params="side y_mul">
+    <!--
+    SERVO TRANS
+    -->
+    <xacro:macro name="servtransmission" params="joint">
+        <transmission name="${joint}_transm">
+            <type>transmission_interface/SimpleTransmission</type>
+            <joint name="${joint}">
+                <hardwareInterface>hardware_interface/PositionJointInterface</hardwareInterface>
+            </joint>
+            <actuator name="${joint}_motor">
+                <hardwareInterface>hardware_interface/PositionActuatorInterface</hardwareInterface>
+            </actuator>
+        </transmission>
+    </xacro:macro>
+    <!--
+    FULL LEG
+    -->
+    <xacro:macro name="bd1_leg" params="side y_mul servo_velocity">
         <!--
         UP
@@ -43,9 +60,12 @@
             </inertial>
         </link>
-        <joint name="up_leg_${side}_j" type="fixed">
+        <joint name="up_leg_${side}_j" type="revolute">
             <parent link="body_link"/>
             <child link="up_leg_${side}_link"/>
             <origin xyz="0 ${y_mul*legs_baseline/2} 0" rpy="0 ${pi/2} 0"/>
+            <limit effort="30" velocity="${servo_velocity}" lower="${-pi/2}" upper="${pi/2}"/>
+            <axis xyz="0 1 0"/>
         </joint>
+        <xacro:servtransmission joint="up_leg_${side}_j"/>
         <!--
         MID
@@ -114,4 +134,11 @@
             <origin xyz="0.15 ${-y_mul*0.0045} 0" rpy="0 ${-pi/2} 0"/>
         </joint>
+        <gazebo reference="feet_${side}_link">
+            <!--<material>Gazebo/Black</material>-->
+            <mu1>20</mu1>
+            <mu2>30</mu2>
+            <!--<dampingFactor>0.05</dampingFactor>-->
+            <!--<kp>10000000000</kp>-->
+        </gazebo>
     </xacro:macro>
 </robot>

Commit message: added legs control service

File: bd1_description/urdf/bd1.xacro (robot description, xacro)
@@ -7,4 +7,7 @@
     <xacro:property name="body_aprox_z" value="0.13"/>
     <xacro:property name="body_mass" value="0.5"/>
+    <xacro:property name="body_shift_x" value="-0.015"/>
+    <xacro:property name="body_shift_y" value="0.0"/>
+    <xacro:property name="body_shift_z" value="0.005"/>
     <xacro:property name="neck_aprox_x" value="0.1"/>
     <xacro:property name="neck_aprox_y" value="0.1"/>
@@ -17,4 +20,7 @@
     <xacro:property name="head_x_offset" value="-0.05"/>
     <xacro:property name="head_z_offset" value="0.1"/>
+    <xacro:property name="head_shift_x" value="0.04"/>
+    <xacro:property name="head_shift_y" value="0.0"/>
+    <xacro:property name="head_shift_z" value="0.07"/>
     <xacro:property name="servo_velocity" value="0.5"/>
     <!--
@@ -37,5 +43,5 @@
         </visual>
         <collision>
-            <origin xyz="-0.015 0 0.005" rpy=" 0 0 0"/>
+            <origin xyz="${body_shift_x} ${body_shift_y} ${body_shift_z}" rpy=" 0 0 0"/>
             <geometry>
                 <box size="${body_aprox_x} ${body_aprox_y} ${body_aprox_z}"/>
@@ -43,4 +49,5 @@
         </collision>
         <inertial>
+            <origin xyz="${body_shift_x} ${body_shift_y} ${body_shift_z}" rpy=" 0 0 0"/>
             <mass value="${body_mass}"/>
             <inertia
@@ -91,5 +98,5 @@
         </visual>
         <collision>
-            <origin xyz="0.04 0 0.07" rpy=" 0 0 0"/>
+            <origin xyz="${head_shift_x} ${head_shift_y} ${head_shift_z}" rpy=" 0 0 0"/>
             <geometry>
                 <box size="${head_aprox_x} ${head_aprox_y} ${head_aprox_z}"/>
@@ -97,4 +104,5 @@
         </collision>
         <inertial>
+            <origin xyz="${head_shift_x} ${head_shift_y} ${head_shift_z}" rpy=" 0 0 0"/>
             <mass value="${head_mass}"/>
             <inertia

File: bd1_description/urdf/bd1_leg.xacro (robot description, xacro)
@@ -6,12 +6,21 @@
     <xacro:property name="up_leg_aprox_z" value="0.12"/>
     <xacro:property name="up_leg_mass" value="0.25"/>
+    <xacro:property name="up_shift_x" value="0.065"/>
+    <xacro:property name="up_shift_y" value="0.03"/>
+    <xacro:property name="up_shift_z" value="0.0"/>
     <xacro:property name="mid_leg_aprox_x" value="0.22"/>
     <xacro:property name="mid_leg_aprox_y" value="0.02"/>
     <xacro:property name="mid_leg_aprox_z" value="0.08"/>
     <xacro:property name="mid_leg_mass" value="0.25"/>
+    <xacro:property name="mid_shift_x" value="0.07"/>
+    <xacro:property name="mid_shift_y" value="0.01"/>
+    <xacro:property name="mid_shift_z" value="0.0"/>
     <xacro:property name="feet_aprox_x" value="0.25"/>
     <xacro:property name="feet_aprox_y" value="0.06"/>
     <xacro:property name="feet_aprox_z" value="0.025"/>
     <xacro:property name="feet_mass" value="0.25"/>
+    <xacro:property name="feet_shift_x" value="0.02"/>
+    <xacro:property name="feet_shift_y" value="0.0"/>
+    <xacro:property name="feet_shift_z" value="-0.065"/>
     <!--
     SERVO TRANS
@@ -46,5 +55,5 @@
             </visual>
             <collision>
-                <origin xyz="0.065 ${y_mul*0.03} 0.0" rpy=" 0 0 0"/>
+                <origin xyz="${up_shift_x} ${y_mul*up_shift_y} ${up_shift_z}" rpy=" 0 0 0"/>
                 <geometry>
                     <box size="${up_leg_aprox_x} ${up_leg_aprox_y} ${up_leg_aprox_z}"/>
@@ -52,4 +61,5 @@
             </collision>
             <inertial>
+                <origin xyz="${up_shift_x} ${y_mul*up_shift_y} ${up_shift_z}" rpy=" 0 0 0"/>
                 <mass value="${up_leg_mass}"/>
                 <inertia
@@ -82,5 +92,5 @@
             </visual>
             <collision>
-                <origin xyz="0.07 ${-y_mul*0.01} 0.0" rpy=" 0 0 0"/>
+                <origin xyz="${mid_shift_x} ${-y_mul*mid_shift_y} ${mid_shift_z}" rpy=" 0 0 0"/>
                 <geometry>
                     <box size="${mid_leg_aprox_x} ${mid_leg_aprox_y} ${mid_leg_aprox_z}"/>
@@ -88,4 +98,5 @@
             </collision>
             <inertial>
+                <origin xyz="${mid_shift_x} ${-y_mul*mid_shift_y} ${mid_shift_z}" rpy=" 0 0 0"/>
                 <mass value="${mid_leg_mass}"/>
                 <inertia
@@ -100,5 +111,5 @@
             <child link="mid_leg_${side}_link"/>
             <origin xyz="0.15 ${y_mul*0.009} 0" rpy="0 0 0"/>
-            <limit effort="30" velocity="${servo_velocity}" lower="${-pi/2}" upper="${pi/2}"/>
+            <limit effort="30" velocity="${servo_velocity*2}" lower="${-pi/2}" upper="${pi/2}"/>
             <axis xyz="0 1 0"/>
         </joint>
@@ -118,5 +129,5 @@
             </visual>
             <collision>
-                <origin xyz="0.02 ${-y_mul*0.0} -0.065" rpy=" 0 0 0"/>
+                <origin xyz="${feet_shift_x} ${-y_mul*feet_shift_y} ${feet_shift_z}" rpy=" 0 0 0"/>
                 <geometry>
                     <box size="${feet_aprox_x} ${feet_aprox_y} ${feet_aprox_z}"/>
@@ -124,4 +135,5 @@
             </collision>
             <inertial>
+                <origin xyz="${feet_shift_x} ${-y_mul*feet_shift_y} ${feet_shift_z}" rpy=" 0 0 0"/>
                 <mass value="${feet_mass}"/>
                 <inertia
@@ -141,6 +153,6 @@
         <gazebo reference="feet_${side}_link">
             <!--<material>Gazebo/Black</material>-->
-            <mu1>20</mu1>
-            <mu2>30</mu2>
+            <mu1>2</mu1>
+            <mu2>5</mu2>
             <!--<dampingFactor>0.05</dampingFactor>-->
             <!--<kp>10000000000</kp>-->

Commit message: changed neck and legs on joint_trajectory_comtrollers

File: bd1_description/urdf/bd1.xacro (robot description, xacro)
@@ -83,5 +83,5 @@
         <axis xyz="0 1 0"/>
     </joint>
-    <xacro:servtransmission joint="neck_j"/>
+    <xacro:servtransmission_v joint="neck_j"/>
     <!--
         HEAD

File: bd1_description/urdf/bd1_leg.xacro (robot description, xacro)
@@ -34,4 +34,15 @@
             <actuator name="${joint}_motor">
                 <hardwareInterface>hardware_interface/PositionActuatorInterface</hardwareInterface>
+            </actuator>
+        </transmission>
+    </xacro:macro>
+    <xacro:macro name="servtransmission_v" params="joint">
+        <transmission name="${joint}_transm">
+            <type>transmission_interface/SimpleTransmission</type>
+            <joint name="${joint}">
+                <hardwareInterface>hardware_interface/VelocityJointInterface</hardwareInterface>
+            </joint>
+            <actuator name="${joint}_motor">
+                <hardwareInterface>hardware_interface/VelocityActuatorInterface</hardwareInterface>
             </actuator>
         </transmission>
@@ -77,5 +88,5 @@
             <axis xyz="0 1 0"/>
         </joint>
-        <xacro:servtransmission joint="up_leg_${side}_j"/>
+        <xacro:servtransmission_v joint="up_leg_${side}_j"/>
         <!--
         MID
@@ -111,8 +122,8 @@
             <child link="mid_leg_${side}_link"/>
             <origin xyz="0.15 ${y_mul*0.009} 0" rpy="0 0 0"/>
-            <limit effort="30" velocity="${servo_velocity*2}" lower="${-pi/2}" upper="${pi/2}"/>
+            <limit effort="30" velocity="${servo_velocity*2}" lower="${-pi}" upper="${pi}"/>
             <axis xyz="0 1 0"/>
         </joint>
-        <xacro:servtransmission joint="mid_leg_${side}_j"/>
+        <xacro:servtransmission_v joint="mid_leg_${side}_j"/>
         <!--
         FEET
@@ -158,5 +169,5 @@
             <!--<kp>10000000000</kp>-->
         </gazebo>
-        <xacro:servtransmission joint="feet_${side}_j"/>
+        <xacro:servtransmission_v joint="feet_${side}_j"/>
     </xacro:macro>
 </robot>

Commit message: added basic moves: strech, deploy, conseal

File: bd1_description/urdf/bd1.xacro (robot description, xacro)
@@ -5,5 +5,5 @@
     <xacro:property name="body_aprox_x" value="0.18"/>
     <xacro:property name="body_aprox_y" value="0.12"/>
-    <xacro:property name="body_aprox_z" value="0.13"/>
+    <xacro:property name="body_aprox_z" value="0.1"/>
     <xacro:property name="body_mass" value="0.5"/>
     <xacro:property name="body_shift_x" value="-0.015"/>
@@ -14,14 +14,16 @@
     <xacro:property name="neck_aprox_z" value="0.1"/>
     <xacro:property name="neck_mass" value="0.01"/>
+    <xacro:property name="neck_shift_x" value="0.03"/>
+    <xacro:property name="neck_shift_y" value="0.0"/>
+    <xacro:property name="neck_shift_z" value="0.04"/>
+    <xacro:property name="neck_len" value="0.07"/>
     <xacro:property name="head_aprox_x" value="0.29"/>
     <xacro:property name="head_aprox_y" value="0.24"/>
-    <xacro:property name="head_aprox_z" value="0.1"/>
+    <xacro:property name="head_aprox_z" value="0.08"/>
     <xacro:property name="head_mass" value="0.5"/>
-    <xacro:property name="head_x_offset" value="-0.05"/>
-    <xacro:property name="head_z_offset" value="0.1"/>
     <xacro:property name="head_shift_x" value="0.04"/>
     <xacro:property name="head_shift_y" value="0.0"/>
     <xacro:property name="head_shift_z" value="0.07"/>
-    <xacro:property name="servo_velocity" value="0.5"/>
+    <xacro:property name="servo_velocity" value="1"/>
     <!--
         BASE
@@ -79,5 +81,5 @@
         <parent link="body_link"/>
         <child link="neck_link"/>
-        <origin xyz="0.02 0 0.02" rpy="0 0 0"/>
+        <origin xyz="${neck_shift_x} ${neck_shift_y} ${neck_shift_z}" rpy="0 0 0"/>
         <limit effort="30" velocity="${servo_velocity}" lower="${-pi/2}" upper="${pi/2}"/>
         <axis xyz="0 1 0"/>
@@ -116,5 +118,5 @@
         <parent link="neck_link"/>
         <child link="head_link"/>
-        <origin xyz="0 0 ${head_z_offset}" rpy="0 0 0"/>
+        <origin xyz="0 0 ${neck_len}" rpy="0 0 0"/>
         <limit effort="30" velocity="${servo_velocity}" lower="${-pi/2}" upper="${pi/2}"/>
         <axis xyz="0 1 0"/>

Commit message: added state and revard service

File: bd1_description/urdf/bd1.xacro (robot description, xacro)
@@ -25,5 +25,5 @@
     <xacro:property name="head_shift_y" value="0.0"/>
     <xacro:property name="head_shift_z" value="0.07"/>
-    <xacro:property name="servo_velocity" value="1"/>
+    <xacro:property name="servo_velocity" value="2"/>
     <!--
         BASE

File: bd1_description/urdf/bd1_leg.xacro (robot description, xacro)
@@ -122,5 +122,5 @@
             <child link="mid_leg_${side}_link"/>
             <origin xyz="0.15 ${y_mul*0.009} 0" rpy="0 0 0"/>
-            <limit effort="30" velocity="${servo_velocity*2}" lower="${-pi}" upper="0"/>
+            <limit effort="30" velocity="${servo_velocity}" lower="${-pi}" upper="0"/>
             <axis xyz="0 1 0"/>
         </joint>
@@ -167,5 +167,5 @@
             <mu2>5</mu2>
             <!--<dampingFactor>0.05</dampingFactor>-->
-            <kp>50000</kp>
+            <kp>20000</kp>
             <kd>1</kd>
         </gazebo>

Commit message: set up DDPG but not tested yet

File: bd1_description/urdf/bd1.xacro (robot description, xacro)
@@ -10,8 +10,8 @@
     <xacro:property name="body_shift_y" value="0.0"/>
     <xacro:property name="body_shift_z" value="0.005"/>
-    <xacro:property name="neck_aprox_x" value="0.1"/>
-    <xacro:property name="neck_aprox_y" value="0.1"/>
+    <xacro:property name="neck_mass" value="0.1"/>
+    <xacro:property name="neck_aprox_x" value="0.02"/>
+    <xacro:property name="neck_aprox_y" value="0.03"/>
     <xacro:property name="neck_aprox_z" value="0.1"/>
-    <xacro:property name="neck_mass" value="0.01"/>
     <xacro:property name="neck_shift_x" value="0.03"/>
     <xacro:property name="neck_shift_y" value="0.0"/>
@@ -69,4 +69,9 @@
     -->
     <link name="neck_link">
+        <visual>
+            <geometry>
+                <mesh filename="file://$(find bd1_description)/mesh/neck_m.dae"/>
+            </geometry>
+        </visual>
         <inertial>
             <mass value="${neck_mass}"/>
@@ -76,4 +81,5 @@
                 izz="${0.08*neck_mass*(neck_aprox_x*neck_aprox_x+neck_aprox_y*neck_aprox_y)}"
             />
+            <origin xyz="0 0 ${head_shift_z/2}" rpy=" 0 0 0"/>
         </inertial>
     </link>

Commit message: new contacts fall detector, DDPG now controlls both legs, but still not very good results

File: bd1_description/urdf/bd1.xacro (robot description, xacro)
@@ -44,5 +44,5 @@
             </material>
         </visual>
-        <collision>
+        <collision name="body_link_collision">
             <origin xyz="${body_shift_x} ${body_shift_y} ${body_shift_z}" rpy=" 0 0 0"/>
             <geometry>

Commit message: now can choose between Trajectory and Velocity controllers, fixed urdf little bit

File: bd1_description/urdf/bd1.xacro (robot description, xacro)
@@ -25,5 +25,9 @@
     <xacro:property name="head_shift_y" value="0.0"/>
     <xacro:property name="head_shift_z" value="0.07"/>
+    <xacro:property name="neck_i_mul" value="10"/>
     <xacro:property name="servo_velocity" value="2"/>
+    <xacro:property name="servo_friction" value="0.3"/>
+    <xacro:property name="servo_effort" value="30"/>
+    <selfCollide>true</selfCollide>
     <!--
         BASE
@@ -77,7 +81,7 @@
             <mass value="${neck_mass}"/>
             <inertia
-                ixx="${0.08*neck_mass*(neck_aprox_y*neck_aprox_y+neck_aprox_z*neck_aprox_z)}" ixy="0" ixz="0"
-                iyy="${0.08*neck_mass*(neck_aprox_x*neck_aprox_x+neck_aprox_z*neck_aprox_z)}" iyz="0"
-                izz="${0.08*neck_mass*(neck_aprox_x*neck_aprox_x+neck_aprox_y*neck_aprox_y)}"
+                ixx="${neck_i_mul*0.08*neck_mass*(neck_aprox_y*neck_aprox_y+neck_aprox_z*neck_aprox_z)}" ixy="0" ixz="0"
+                iyy="${neck_i_mul*0.08*neck_mass*(neck_aprox_x*neck_aprox_x+neck_aprox_z*neck_aprox_z)}" iyz="0"
+                izz="${neck_i_mul*0.08*neck_mass*(neck_aprox_x*neck_aprox_x+neck_aprox_y*neck_aprox_y)}"
             />
             <origin xyz="0 0 ${head_shift_z/2}" rpy=" 0 0 0"/>
@@ -88,6 +92,7 @@
         <child link="neck_link"/>
         <origin xyz="${neck_shift_x} ${neck_shift_y} ${neck_shift_z}" rpy="0 0 0"/>
-        <limit effort="30" velocity="${servo_velocity}" lower="${-pi/2}" upper="${pi/2}"/>
+        <limit effort="${servo_effort}" velocity="${servo_velocity}" lower="-1.5" upper="1.5"/>
         <axis xyz="0 1 0"/>
+        <dynamics damping="${servo_friction}"/>
     </joint>
     <xacro:servtransmission_v joint="neck_j"/>
@@ -125,6 +130,7 @@
         <child link="head_link"/>
         <origin xyz="0 0 ${neck_len}" rpy="0 0 0"/>
-        <limit effort="30" velocity="${servo_velocity}" lower="${-pi/2}" upper="${pi/2}"/>
+        <limit effort="${servo_effort}" velocity="${servo_velocity}" lower="-1.5" upper="1.5"/>
         <axis xyz="0 1 0"/>
+        <dynamics damping="${servo_friction}"/>
     </joint>
     <xacro:servtransmission_v joint="head_j"/>
@@ -132,5 +138,5 @@
         LEGS
     -->
-    <xacro:bd1_leg side="r" y_mul="-1" servo_velocity="${servo_velocity}"/>
-    <xacro:bd1_leg side="l" y_mul="1" servo_velocity="${servo_velocity}"/>
+    <xacro:bd1_leg side="r" y_mul="-1" servo_velocity="${servo_velocity}" servo_effort="${servo_effort}"/>
+    <xacro:bd1_leg side="l" y_mul="1" servo_velocity="${servo_velocity}" servo_effort="${servo_effort}"/>
 </robot>

File: bd1_description/urdf/bd1_leg.xacro (robot description, xacro)
@@ -51,5 +51,5 @@
     FULL LEG
     -->
-    <xacro:macro name="bd1_leg" params="side y_mul servo_velocity">
+    <xacro:macro name="bd1_leg" params="side y_mul servo_velocity servo_effort">
         <!--
         UP
@@ -85,5 +85,5 @@
             <child link="up_leg_${side}_link"/>
             <origin xyz="0 ${y_mul*legs_baseline/2} 0" rpy="0 ${pi/2} 0"/>
-            <limit effort="30" velocity="${servo_velocity}" lower="${-pi/2}" upper="${pi/2}"/>
+            <limit effort="${servo_effort}" velocity="${servo_velocity}" lower="${-pi/2}" upper="1.5"/>
             <axis xyz="0 1 0"/>
         </joint>
@@ -122,5 +122,5 @@
             <child link="mid_leg_${side}_link"/>
             <origin xyz="0.15 ${y_mul*0.009} 0" rpy="0 0 0"/>
-            <limit effort="30" velocity="${servo_velocity}" lower="${-pi}" upper="0"/>
+            <limit effort="${servo_effort}" velocity="${servo_velocity}" lower="-3" upper="0"/>
             <axis xyz="0 1 0"/>
         </joint>
@@ -159,5 +159,5 @@
             <child link="feet_${side}_link"/>
             <origin xyz="0.15 ${-y_mul*0.0045} 0" rpy="0 ${-pi/2} 0"/>
-            <limit effort="30" velocity="${servo_velocity}" lower="${-pi/2}" upper="${pi/2}"/>
+            <limit effort="${servo_effort}" velocity="${servo_velocity}" lower="${-pi/2}" upper="1.5"/>
             <axis xyz="0 1 0"/>
         </joint>

Commit message: added new interface new Rl method

File: bd1_description/urdf/bd1.xacro (robot description, xacro)
@@ -91,6 +91,6 @@
         <parent link="body_link"/>
         <child link="neck_link"/>
-        <origin xyz="${neck_shift_x} ${neck_shift_y} ${neck_shift_z}" rpy="0 0 0"/>
-        <limit effort="${servo_effort}" velocity="${servo_velocity}" lower="-1.5" upper="1.5"/>
+        <origin xyz="${neck_shift_x} ${neck_shift_y} ${neck_shift_z}" rpy="0 -1.5 0"/>
+        <limit effort="${servo_effort}" velocity="${servo_velocity}" lower="0" upper="${pi}"/>
         <axis xyz="0 1 0"/>
         <dynamics damping="${servo_friction}"/>
@@ -129,6 +129,6 @@
         <parent link="neck_link"/>
         <child link="head_link"/>
-        <origin xyz="0 0 ${neck_len}" rpy="0 0 0"/>
-        <limit effort="${servo_effort}" velocity="${servo_velocity}" lower="-1.5" upper="1.5"/>
+        <origin xyz="0 0 ${neck_len}" rpy="0 1.5 0"/>
+        <limit effort="${servo_effort}" velocity="${servo_velocity}" lower="0" upper="${pi}"/>
         <axis xyz="0 1 0"/>
         <dynamics damping="${servo_friction}"/>
