Commit message: added universal gazebo interface, universal PPO trainer and manual velocity controll via dynamic reconf

File: bd1_description/urdf/bd1.xacro (robot description, xacro)
@@ -28,5 +28,5 @@
     <xacro:property name="servo_velocity" value="2"/>
     <xacro:property name="servo_friction" value="0.3"/>
-    <xacro:property name="servo_effort" value="30"/>
+    <xacro:property name="servo_effort" value="60"/>
     <selfCollide>true</selfCollide>
     <!--
@@ -130,5 +130,5 @@
         <child link="head_link"/>
         <origin xyz="0 0 ${neck_len}" rpy="0 1.5 0"/>
-        <limit effort="${servo_effort}" velocity="${servo_velocity}" lower="0" upper="${pi}"/>
+        <limit effort="${servo_effort}" velocity="${servo_velocity}" lower="${-pi}" upper="0"/>
         <axis xyz="0 1 0"/>
         <dynamics damping="${servo_friction}"/>

File: bd1_description/urdf/bd1_leg.xacro (robot description, xacro)
@@ -167,5 +167,5 @@
             <mu2>5</mu2>
             <!--<dampingFactor>0.05</dampingFactor>-->
-            <kp>20000</kp>
+            <kp>100000</kp>
             <kd>1</kd>
         </gazebo>

Commit message: added effort controllers too

File: bd1_description/urdf/bd1.xacro (robot description, xacro)
@@ -1,6 +1,8 @@
 <?xml version="1.0"?>
 <robot xmlns:xacro="http://www.ros.org/wiki/xacro" name="BD1" >
+    <xacro:arg name="servo_control" default="VEL"/>
     <xacro:include filename="$(find bd1_description)/urdf/bd1_leg.xacro"/>
     <xacro:include filename="$(find bd1_description)/urdf/bd1.gazebo"/>
+    <xacro:include filename="$(find bd1_description)/urdf/transmission_$(arg servo_control).xacro"/>
     <xacro:property name="body_aprox_x" value="0.18"/>
     <xacro:property name="body_aprox_y" value="0.12"/>
@@ -28,5 +30,5 @@
     <xacro:property name="servo_velocity" value="2"/>
     <xacro:property name="servo_friction" value="0.3"/>
-    <xacro:property name="servo_effort" value="60"/>
+    <xacro:property name="servo_effort" value="30"/>
     <selfCollide>true</selfCollide>
     <!--
@@ -96,5 +98,5 @@
         <dynamics damping="${servo_friction}"/>
     </joint>
-    <xacro:servtransmission_v joint="neck_j"/>
+    <xacro:servtransmission joint="neck_j"/>
     <!--
         HEAD
@@ -134,5 +136,5 @@
         <dynamics damping="${servo_friction}"/>
     </joint>
-    <xacro:servtransmission_v joint="head_j"/>
+    <xacro:servtransmission joint="head_j"/>
     <!--
         LEGS

File: bd1_description/urdf/bd1_leg.xacro (robot description, xacro)
@@ -23,29 +23,5 @@
     <xacro:property name="feet_shift_y" value="0.0"/>
     <xacro:property name="feet_shift_z" value="-0.065"/>
-    <!--
-    SERVO TRANS
-    -->
-    <xacro:macro name="servtransmission" params="joint">
-        <transmission name="${joint}_transm">
-            <type>transmission_interface/SimpleTransmission</type>
-            <joint name="${joint}">
-                <hardwareInterface>hardware_interface/PositionJointInterface</hardwareInterface>
-            </joint>
-            <actuator name="${joint}_motor">
-                <hardwareInterface>hardware_interface/PositionActuatorInterface</hardwareInterface>
-            </actuator>
-        </transmission>
-    </xacro:macro>
-    <xacro:macro name="servtransmission_v" params="joint">
-        <transmission name="${joint}_transm">
-            <type>transmission_interface/SimpleTransmission</type>
-            <joint name="${joint}">
-                <hardwareInterface>hardware_interface/VelocityJointInterface</hardwareInterface>
-            </joint>
-            <actuator name="${joint}_motor">
-                <hardwareInterface>hardware_interface/VelocityActuatorInterface</hardwareInterface>
-            </actuator>
-        </transmission>
-    </xacro:macro>
+    <xacro:include filename="$(find bd1_description)/urdf/transmission_$(arg servo_control).xacro"/>
     <!--
     FULL LEG
@@ -88,5 +64,5 @@
             <axis xyz="0 1 0"/>
         </joint>
-        <xacro:servtransmission_v joint="up_leg_${side}_j"/>
+        <xacro:servtransmission joint="up_leg_${side}_j"/>
         <!--
         MID
@@ -125,5 +101,5 @@
             <axis xyz="0 1 0"/>
         </joint>
-        <xacro:servtransmission_v joint="mid_leg_${side}_j"/>
+        <xacro:servtransmission joint="mid_leg_${side}_j"/>
         <!--
         FEET
@@ -170,5 +146,5 @@
             <kd>1</kd>
         </gazebo>
-        <xacro:servtransmission_v joint="feet_${side}_j"/>
+        <xacro:servtransmission joint="feet_${side}_j"/>
     </xacro:macro>
 </robot>

Commit message: fixed reset

File: bd1_description/urdf/bd1.xacro (robot description, xacro)
@@ -93,7 +93,7 @@
         <parent link="body_link"/>
         <child link="neck_link"/>
-        <origin xyz="${neck_shift_x} ${neck_shift_y} ${neck_shift_z}" rpy="0 -1.5 0"/>
-        <limit effort="${servo_effort}" velocity="${servo_velocity}" lower="0" upper="${pi}"/>
-        <axis xyz="0 1 0"/>
+        <origin xyz="${neck_shift_x} ${neck_shift_y} ${neck_shift_z}" rpy="0 0 0"/>
+        <limit effort="${servo_effort}" velocity="${servo_velocity}" lower="${-pi/2}" upper="${pi/2}"/>
+        <axis xyz="0 -1 0"/>
         <dynamics damping="${servo_friction}"/>
     </joint>
@@ -131,6 +131,6 @@
         <parent link="neck_link"/>
         <child link="head_link"/>
-        <origin xyz="0 0 ${neck_len}" rpy="0 1.5 0"/>
-        <limit effort="${servo_effort}" velocity="${servo_velocity}" lower="${-pi}" upper="0"/>
+        <origin xyz="0 0 ${neck_len}" rpy="0 0 0"/>
+        <limit effort="${servo_effort}" velocity="${servo_velocity}" lower="0" upper="${pi/2}"/>
         <axis xyz="0 1 0"/>
         <dynamics damping="${servo_friction}"/>

File: bd1_description/urdf/bd1_leg.xacro (robot description, xacro)
@@ -68,7 +68,7 @@
             <parent link="body_link"/>
             <child link="hip_${side}_link"/>
-            <origin xyz="0 ${y_mul*legs_baseline/2} 0" rpy="0 ${pi/2+1.5} 0"/>
-            <limit effort="${servo_effort}" velocity="${servo_velocity}" lower="${-pi}0" upper="0"/>
-            <axis xyz="0 1 0"/>
+            <origin xyz="0 ${y_mul*legs_baseline/2} 0" rpy="0 ${pi/2} 0"/>
+            <limit effort="${servo_effort}" velocity="${servo_velocity}" lower="${-pi/2}" upper="0"/>
+            <axis xyz="0 -1 0"/>
             <!--<dynamics damping="${servo_friction}"/>-->
         </joint>
@@ -106,7 +106,7 @@
             <parent link="hip_${side}_link"/>
             <child link="knee_${side}_link"/>
-            <origin xyz="0.15 ${y_mul*0.009} 0" rpy="0 -3 0"/>
+            <origin xyz="0.15 ${y_mul*0.009} 0" rpy="0 0 0"/>
             <limit effort="${servo_effort}" velocity="${servo_velocity}" lower="0" upper="${pi}"/>
-            <axis xyz="0 1 0"/>
+            <axis xyz="0 -1 0"/>
             <!--<dynamics damping="${servo_friction}"/>-->
         </joint>
@@ -144,6 +144,6 @@
             <parent link="knee_${side}_link"/>
             <child link="foot_${side}_link"/>
-            <origin xyz="0.15 ${-y_mul*0.0045} 0" rpy="0 0 0"/>
-            <limit effort="${servo_effort}" velocity="${servo_velocity}" lower="${-pi}" upper="0"/>
+            <origin xyz="0.15 ${-y_mul*0.0045} 0" rpy="0 ${-pi/2} 0"/>
+            <limit effort="${servo_effort}" velocity="${servo_velocity}" lower="${-pi/2}" upper="${pi/2}"/>
             <axis xyz="0 1 0"/>
             <!--<dynamics damping="${servo_friction}"/>-->

Commit message: Set effort limit as said in AX-12 spec

File: bd1_description/urdf/bd1.xacro (robot description, xacro)
@@ -30,5 +30,5 @@
     <xacro:property name="servo_velocity" value="2"/>
     <xacro:property name="servo_friction" value="0.3"/>
-    <xacro:property name="servo_effort" value="30"/>
+    <xacro:property name="servo_effort" value="1.5"/>
     <selfCollide>true</selfCollide>
     <!--

Commit message: her shows some works

File: bd1_description/urdf/bd1.xacro (robot description, xacro)
@@ -30,5 +30,5 @@
     <xacro:property name="servo_velocity" value="2"/>
     <xacro:property name="servo_friction" value="0.3"/>
-    <xacro:property name="servo_effort" value="1.5"/>
+    <xacro:property name="servo_effort" value="30"/>
     <selfCollide>true</selfCollide>
     <!--
